File: HB-UNI-Sensor1-CO2_SCD30/PCB/Modification_of_TomMajors_Smarthome/HB-UNI-Sensor1-CO2_SCD30/HB-UNI-SEN-BATT_mod/HB-UNI-SEN-BATT_mod.sch (KiCad schematic (older format))
At the start: 35 parts, among them J10 Conn_01x02-conn, J11 Conn_01x04-conn, J12 Conn_01x04-conn, J13 Conn_01x04-conn, J14 Conn_01x04-conn, J4 Conn_01x02-conn, J5 GS2-conn, J6 Conn_01x04-conn, J7 Conn_01x02-conn, J8 Conn_01x02-conn, J9 Conn_01x02-conn, Q1 BC327, SW2 SW_DIP_x01-switches, U1 CC1101-RESCUE-HB-UNI-SEN-BATT, U2 ArduinoProMini

Commit message: Release V1.0
Parts:
- C1: value CP -> 10u
- C2: value CP -> 470u
- R10, R11, R4, R5: value R -> 10k
- R2: value R -> 470
- R3: value R -> 100
- R6, R7, R8, R9: value R -> 47k 1%
Changed lines of the file:
@@
 P 6850 5350
 F 0 "J9" H 6850 5450 50  0000 C CNN
-F 1 "Conn_01x02-conn" H 6850 5150 50  0000 C CNN
+F 1 "Conn_01x02-conn" H 6750 5000 50  0000 C CNN
 F 2 "Pin_Headers:Pin_Header_Straight_1x02_Pitch2.54mm" H 6850 5350 50  0001 C CNN
 F 3 "" H 6850 5350 50  0001 C CNN
@@
 P 4700 4050
 F 0 "R2" V 4780 4050 50  0000 C CNN
-F 1 "R" V 4700 4050 50  0000 C CNN
+F 1 "470" V 4700 4050 50  0000 C CNN
 F 2 "Resistors_THT:R_Axial_DIN0207_L6.3mm_D2.5mm_P2.54mm_Vertical" V 4630 4050 50  0001 C CNN
 F 3 "~" H 4700 4050 50  0001 C CNN
@@
 P 6800 1500
 F 0 "C1" H 6825 1600 50  0000 L CNN
-F 1 "CP" H 6825 1400 50  0000 L CNN
+F 1 "10u" H 6825 1400 50  0000 L CNN
 F 2 "Capacitors_THT:CP_Radial_D4.0mm_P1.50mm" H 6838 1350 50  0001 C CNN
 F 3 "~" H 6800 1500 50  0001 C CNN
@@
 P 10950 1550
 F 0 "R10" V 11030 1550 50  0000 C CNN
-F 1 "R" V 10950 1550 50  0000 C CNN
+F 1 "10k" V 10950 1550 50  0000 C CNN
 F 2 "Resistors_THT:R_Axial_DIN0207_L6.3mm_D2.5mm_P2.54mm_Vertical" V 10880 1550 50  0001 C CNN
 F 3 "~" H 10950 1550 50  0001 C CNN
@@
 P 10950 1750
 F 0 "R11" V 11030 1750 50  0000 C CNN
-F 1 "R" V 10950 1750 50  0000 C CNN
+F 1 "10k" V 10950 1750 50  0000 C CNN
 F 2 "Resistors_THT:R_Axial_DIN0207_L6.3mm_D2.5mm_P2.54mm_Vertical" V 10880 1750 50  0001 C CNN
 F 3 "~" H 10950 1750 50  0001 C CNN
@@
 P 8750 1100
 F 0 "C2" H 8868 1146 50  0000 L CNN
-F 1 "CP" H 8400 1100 50  0000 L CNN
+F 1 "470u" H 8400 1100 50  0000 L CNN
 F 2 "" H 8788 950 50  0001 C CNN
 F 3 "~" H 8750 1100 50  0001 C CNN
@@
 P 6050 1350
 F 0 "R4" H 6120 1396 50  0000 L CNN
-F 1 "R" H 6120 1305 50  0000 L CNN
+F 1 "10k" H 6120 1305 50  0000 L CNN
 F 2 "" V 5980 1350 50  0001 C CNN
 F 3 "~" H 6050 1350 50  0001 C CNN
@@
 P 6050 1800
 F 0 "R5" H 6120 1846 50  0000 L CNN
-F 1 "R" H 6120 1755 50  0000 L CNN
+F 1 "10k" H 6120 1755 50  0000 L CNN
 F 2 "" V 5980 1800 50  0001 C CNN
 F 3 "~" H 6050 1800 50  0001 C CNN
@@
 P 5650 1900
 F 0 "R3" H 5720 1946 50  0000 L CNN
-F 1 "R" H 5720 1855 50  0000 L CNN
+F 1 "100" H 5720 1855 50  0000 L CNN
 F 2 "" V 5580 1900 50  0001 C CNN
 F 3 "~" H 5650 1900 50  0001 C CNN
@@
 P 7250 4950
 F 0 "R6" H 7250 4800 50  0000 L CNN
-F 1 "R" V 7150 4850 50  0000 L CNN
+F 1 "47k 1%" V 7150 4850 50  0000 L CNN
 F 2 "" V 7180 4950 50  0001 C CNN
 F 3 "~" H 7250 4950 50  0001 C CNN
@@
 P 7550 4950
 F 0 "R8" H 7550 4800 50  0000 L CNN
-F 1 "R" V 7450 4850 50  0000 L CNN
+F 1 "47k 1%" V 7450 4850 50  0000 L CNN
 F 2 "" V 7480 4950 50  0001 C CNN
 F 3 "~" H 7550 4950 50  0001 C CNN
@@
 P 7550 5500
 F 0 "R9" H 7550 5350 50  0000 L CNN
-F 1 "R" V 7450 5450 50  0000 L CNN
+F 1 "47k 1%" V 7450 5450 50  0000 L CNN
 F 2 "" V 7480 5500 50  0001 C CNN
 F 3 "~" H 7550 5500 50  0001 C CNN
@@
 P 7250 5500
 F 0 "R7" H 7250 5350 50  0000 L CNN
-F 1 "R" V 7150 5400 50  0000 L CNN
+F 1 "47k 1%" V 7150 5400 50  0000 L CNN
 F 2 "" V 7180 5500 50  0001 C CNN
 F 3 "~" H 7250 5500 50  0001 C CNN
