File: HB-UNI-Sensor1-CO2_SCD30/PCB/Modification_of_Alexander_Reinerts_PCB/HB-UNI-Sensor1-CO2_SCD30/HB-UNI-SEN-BATT_mod/HB-UNI-SEN-BATT_mod.sch (KiCad schematic (older format))
At the start: 35 parts, among them J10 Conn_01x02-conn, J11 Conn_01x04-conn, J12 Conn_01x04-conn, J13 Conn_01x04-conn, J14 Conn_01x04-conn, J4 Conn_01x02-conn, J5 GS2-conn, J6 Conn_01x04-conn, J7 Conn_01x02-conn, J8 Conn_01x02-conn, J9 Conn_01x02-conn, Q1 BC327, SW2 SW_DIP_x01-switches, U1 CC1101-RESCUE-HB-UNI-SEN-BATT, U2 ArduinoProMini

Commit message: Added some comments to the KiCAD schematics
Other:
- note added: "A 470 uF decoupling capacitor attached to the I2C sockets has been removed !"
- note added: "C2 has been added on 6th Sept 2020\n"
Changed lines of the file:
@@
 	4350 1650 4200 1650
 Connection ~ 4200 1650
+Text Notes 3400 1750 0    50   ~ 0
+C2 has been added on 6th Sept 2020\n
+Text Notes 8100 1200 0    50   ~ 0
+A 470 uF decoupling capacitor attached to the I2C sockets has been removed !
 $EndSCHEMATC
